File: control_board/control_board.sch (KiCad schematic (older format))
At the start: 40 parts, among them J1 Conn_01x08_Male, K1 G5Q-1A, Q1 Q_NPN_BEC, U1 MC78M05_TO252, U2 TSR_1-24120, U3 74LS02, U4 74LS02, U5 Conn_01x08_Male

Commit message: Via & trace tweaks
Connections:
- net GND: now also RN1.2 (R2.1)
- no-connect marks 17 -> 16
Changed lines of the file:
@@
 	1    0    0    -1
 $EndComp
-NoConn ~ 7600 4350
 Text Notes 6500 4650 0    50   ~ 0
 RN1 -> 1k\nRN2 -> 1k\nRN3 -> 330
@@
 	1    0    0    -1
 $EndComp
+$Comp
+L power:GND #PWR?
+U 1 1 6029FF95
+P 7600 4350
+F 0 "#PWR?" H 7600 4100 50  0001 C CNN
+F 1 "GND" H 7605 4177 50  0000 C CNN
+F 2 "" H 7600 4350 50  0001 C CNN
+F 3 "" H 7600 4350 50  0001 C CNN
+	1    7600 4350
+	-1   0    0    1
+$EndComp
 $EndSCHEMATC
